Commit message: Update crb15000_10_152_macro.xacro

File: abb_crb15000_support/urdf/crb15000_10_152_macro.xacro (robot description, xacro)
@@ -46,10 +46,10 @@
       <collision>
         <geometry>
-          <mesh filename="package://abb_crb15000_support/meshes/crb15000_5_95/collision/link_3.stl"/>
+          <mesh filename="package://abb_crb15000_support/meshes/crb15000_10_152/collision/link_3.stl"/>
         </geometry>
       </collision>
       <visual>
         <geometry>
-          <mesh filename="package://abb_crb15000_support/meshes/crb15000_5_95/visual/link_3.stl"/>
+          <mesh filename="package://abb_crb15000_support/meshes/crb15000_10_152/visual/link_3.stl"/>
         </geometry>
         <xacro:material_abb_dark_gray />
@@ -72,10 +72,10 @@
       <collision>
         <geometry>
-          <mesh filename="package://abb_crb15000_support/meshes/crb15000_5_95/collision/link_5.stl"/>
+          <mesh filename="package://abb_crb15000_support/meshes/crb15000_10_152/collision/link_5.stl"/>
         </geometry>
       </collision>
       <visual>
         <geometry>
-          <mesh filename="package://abb_crb15000_support/meshes/crb15000_5_95/visual/link_5.stl"/>
+          <mesh filename="package://abb_crb15000_support/meshes/crb15000_10_152/visual/link_5.stl"/>
         </geometry>
         <xacro:material_abb_graphite_white />
@@ -85,10 +85,10 @@
       <collision>
         <geometry>
-          <mesh filename="package://abb_crb15000_support/meshes/crb15000_5_95/collision/link_6.stl"/>
+          <mesh filename="package://abb_crb15000_support/meshes/crb15000_10_152/collision/link_6.stl"/>
         </geometry>
       </collision>
       <visual>
         <geometry>
-          <mesh filename="package://abb_crb15000_support/meshes/crb15000_5_95/visual/link_6.stl"/>
+          <mesh filename="package://abb_crb15000_support/meshes/crb15000_10_152/visual/link_6.stl"/>
         </geometry>
         <xacro:material_abb_gray_white />
